Commit message: changed robot description because it was loading some wrong meshes and non existant files

File: robots/hsrb4s.urdf (robot description, URDF)
Before this commit: robot hsrb, 45 links, 44 joints
Links:
- link torso_lift_link: geometry collision mesh filename=package://hsr_meshes/meshes/torso_v0/torso.stl; visual mesh filename=package://hsr_meshes/meshes/torso_v0/torso_light.dae

File: urdf/sensors/rgbd_sensor.urdf.xacro (robot description, xacro)
@@ -62,5 +62,4 @@
             <child link="${prefix}_${sensor_name}_gazebo_frame"/>
         </joint>
-        `
         <link name="${prefix}_${sensor_name}_gazebo_frame"></link>
         <xacro:rgbd_sensor_gazebo
